Commit message: feat(burger_description): Gen3 de 6 GDL con módulo de visión; taller URDF/TF y su formato ABET
En main los URDF seguían en 7 GDL: la re-vendorización a 6 GDL estaba en la
rama claude/todo-burger-description-6dof sin fusionar. Este cambio la
incorpora (merge anterior) y la completa:

- scripts/revendorizar_gen3_6dof.py --vision: brazalete con visión y los
  frames oficiales gen3_camera_link, gen3_camera_color_frame y
  gen3_camera_depth_frame bajo gen3_end_effector_link (macro de Kinova
  @ b2aa46b). El script regenera además la copia del visor web
  visual/burger_delivery_gen3.urdf, que también estaba en 7 GDL; se
  eliminan las mallas de 7 GDL y la de bracelet_no_vision que ya no usa
  ningún URDF.
- TALLER_URDF_TF.md: pinza Robotiq 2F-85 (1 junta actuada y 5 mimic) y
  nueva §11 sobre la cámara de muñeca: marco de cuerpo frente a marco
  óptico, pose de la cámara en la pose cero, transformar un punto del
  marco óptico a gen3_base_link a mano y con TF2, y el eslabón
  end_effector_link -> camera_link que falta en el robot real porque el
  driver no carga vision:=true. Es lo que necesita la Ruta B del Lab IA 01.
- PLANTILLA_EVIDENCIA_ABET_TALLER_URDF_TF v1.1 (md, json y docx): E3 y
  C1 sin la referencia a 7 GDL, nueva evidencia E7 de la cadena de la
  cámara (las orales pasan a E9-E12) y C2 incluye la cámara.
- Guía IA 01 (Ruta B), README del paquete, visor web, arquitectura,
  INSTALACION_KORTEX, ejercicio de turnos, monitor de red y TODO.md al día.

Co-Authored-By: Claude Opus 5.5 <noreply@anthropic.com>
Claude-Session: https://claude.ai/code/session_01A4jArrxa1RLtDdQTQFnPXP

File: burger_description/urdf/burger_delivery_gen3.urdf (robot description, URDF)
Before this commit: robot burger_delivery_gen3, 42 links, 41 joints
Links:
- added link gen3_camera_color_frame
- added link gen3_camera_depth_frame
- added link gen3_camera_link
- link gen3_bracelet_link: mass 0.364 -> 0.5
Joints:
- added joint gen3_camera_module: type fixed, parent gen3_end_effector_link, child gen3_camera_link, origin xyz=0 0.05639 -0.00305 rpy=3.14159265358979 3.14159265358979 0
- added joint gen3_color_module: type fixed, parent gen3_end_effector_link, child gen3_camera_color_frame, origin xyz=0 0.05639 -0.00305 rpy=3.14159265358979 3.14159265358979 0
- added joint gen3_depth_module: type fixed, parent gen3_end_effector_link, child gen3_camera_depth_frame, origin xyz=0.0275 0.066 -0.00305 rpy=3.14159265358979 3.14159265358979 0

File: burger_description/urdf/delivery_scene_fixed.urdf (robot description, URDF)
Before this commit: robot burger_delivery_scene, 39 links, 38 joints
Links:
- added link gen3_camera_color_frame
- added link gen3_camera_depth_frame
- added link gen3_camera_link
- link gen3_bracelet_link: mass 0.364 -> 0.5
Joints:
- added joint gen3_camera_module: type fixed, parent gen3_end_effector_link, child gen3_camera_link, origin xyz=0 0.05639 -0.00305 rpy=3.14159265358979 3.14159265358979 0
- added joint gen3_color_module: type fixed, parent gen3_end_effector_link, child gen3_camera_color_frame, origin xyz=0 0.05639 -0.00305 rpy=3.14159265358979 3.14159265358979 0
- added joint gen3_depth_module: type fixed, parent gen3_end_effector_link, child gen3_camera_depth_frame, origin xyz=0.0275 0.066 -0.00305 rpy=3.14159265358979 3.14159265358979 0

File: visual/burger_delivery_gen3.urdf (robot description, URDF)
Before this commit: robot burger_delivery_gen3, 43 links, 42 joints
Links:
- removed link gen3_half_arm_1_link
- removed link gen3_half_arm_2_link
- added link gen3_bicep_link, mass 1.262; collision mesh filename=vendor/kortex_description/arms/gen3/6dof/meshes/bicep_link.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; visual mesh filename=vendor/kortex_description/arms/gen3/6dof/meshes/bicep_link.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
- added link gen3_camera_color_frame
- added link gen3_camera_depth_frame
- added link gen3_camera_link
- link gen3_base_link: geometry collision mesh filename=vendor/kortex_description/arms/gen3/6dof/meshes/base_link.S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; visual mesh filename=vendor/kortex_description/arms/gen3/6dof/meshes/base_link.S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
- link gen3_bracelet_link: mass 0.364 -> 0.5; geometry collision mesh filename=vendor/kortex_description/arms/gen3/6dof/meshes/bracelet_wi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; visual mesh filename=vendor/kortex_description/arms/gen3/6dof/meshes/bracelet_wi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
- link gen3_forearm_link: mass 0.9302 -> 0.93; geometry collision mesh filename=vendor/kortex_description/arms/gen3/6dof/meshes/forearm_lin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; visual mesh filename=vendor/kortex_description/arms/gen3/6dof/meshes/forearm_lin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
- link gen3_robotiq_85_base_link: geometry collision mesh filename=vendor/robotiq_description/meshes/collision/2f_85/robotiq_b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; visual mesh filename=vendor/robotiq_description/meshes/visual/2f_85/robotiq_base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
- link gen3_robotiq_85_left_finger_link: geometry collision mesh filename=vendor/robotiq_description/meshes/collision/2f_85/left_fing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; visual mesh filename=vendor/robotiq_description/meshes/visual/2f_85/left_finger.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
- link gen3_robotiq_85_left_finger_tip_link: geometry collision mesh filename=vendor/robotiq_description/meshes/collision/2f_85/left_fing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; visual mesh filename=vendor/robotiq_description/meshes/visual/2f_85/left_finger_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
- link gen3_robotiq_85_left_inner_knuckle_link: geometry collision mesh filename=vendor/robotiq_description/meshes/collision/2f_85/left_inne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; visual mesh filename=vendor/robotiq_description/meshes/visual/2f_85/left_inner_k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
- link gen3_robotiq_85_left_knuckle_link: geometry collision mesh filename=vendor/robotiq_description/meshes/collision/2f_85/left_knuc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; visual mesh filename=vendor/robotiq_description/meshes/visual/2f_85/left_knuckle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
- link gen3_robotiq_85_right_finger_link: geometry collision mesh filename=vendor/robotiq_description/meshes/collision/2f_85/right_fin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; visual mesh filename=vendor/robotiq_description/meshes/visual/2f_85/right_finger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
- link gen3_robotiq_85_right_finger_tip_link: geometry collision mesh filename=vendor/robotiq_description/meshes/collision/2f_85/right_fin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; visual mesh filename=vendor/robotiq_description/meshes/visual/2f_85/right_finger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
- link gen3_robotiq_85_right_inner_knuckle_link: geometry collision mesh filename=vendor/robotiq_description/meshes/collision/2f_85/right_inn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; visual mesh filename=vendor/robotiq_description/meshes/visual/2f_85/right_inner_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
- link gen3_robotiq_85_right_knuckle_link: geometry collision mesh filename=vendor/robotiq_description/meshes/collision/2f_85/right_knu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; visual mesh filename=vendor/robotiq_description/meshes/visual/2f_85/right_knuckl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
- link gen3_shoulder_link: mass 1.3773 -> 1.377; geometry collision mesh filename=vendor/kortex_description/arms/gen3/6dof/meshes/shoulder_li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; visual mesh filename=vendor/kortex_description/arms/gen3/6dof/meshes/shoulder_li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
- link gen3_spherical_wrist_1_link: geometry collision mesh filename=vendor/kortex_description/arms/gen3/6dof/meshes/spherical_w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; visual mesh filename=vendor/kortex_description/arms/gen3/6dof/meshes/spherical_w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
- link gen3_spherical_wrist_2_link: mass 0.6781 -> 0.678; geometry collision mesh filename=vendor/kortex_description/arms/gen3/6dof/meshes/spherical_w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; visual mesh filename=vendor/kortex_description/arms/gen3/6dof/meshes/spherical_w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
- link wrist_camera_mount_link: geometry collision box size=0.04 0.08 0.06; visual box size=0.04 0.08 0.06
Joints:
- removed joint gen3_joint_7
- added joint gen3_camera_module: type fixed, parent gen3_end_effector_link, child gen3_camera_link, origin xyz=0 0.05639 -0.00305 rpy=3.14159265358979 3.14159265358979 0
- added joint gen3_color_module: type fixed, parent gen3_end_effector_link, child gen3_camera_color_frame, origin xyz=0 0.05639 -0.00305 rpy=3.14159265358979 3.14159265358979 0
- added joint gen3_depth_module: type fixed, parent gen3_end_effector_link, child gen3_camera_depth_frame, origin xyz=0.0275 0.066 -0.00305 rpy=3.14159265358979 3.14159265358979 0
- joint gen3_end_effector: origin xyz=0 0 -0.0615250000000001 rpy=3.14159265358979 1.09937075168372E-32 0 -> xyz=0 0 -0.0615250000000001 rpy=3.14159265358979 1.09937075168372E-32 3.14159265358979
- joint gen3_joint_1: origin xyz=0 0 0.15643 rpy=3.1416 2.7629E-18 -4.9305E-36 -> xyz=0 0 0.15643 rpy=-3.1416 0.0 0.0
- joint gen3_joint_2: child gen3_half_arm_1_link -> gen3_bicep_link; limit lower=-2.41 upper=2.41 effort=39 velocity=1.3963 -> lower=-2.24 upper=2.24 effort=39 velocity=1.3963; origin xyz=0 0.005375 -0.12838 rpy=1.5708 2.1343E-17 -1.1102E-16 -> xyz=0 0.005375 -0.12838 rpy=1.5708 0.0 0.0
- joint gen3_joint_3: child gen3_half_arm_2_link -> gen3_forearm_link; limit effort=39 velocity=1.3963 -> lower=-2.57 upper=2.57 effort=39 velocity=1.3963; origin xyz=0 -0.21038 -0.006375 rpy=-1.5708 1.2326E-32 -2.9122E-16 -> xyz=0 -0.41 0 rpy=3.1416 0 0; parent gen3_half_arm_1_link -> gen3_bicep_link; type continuous -> revolute
- joint gen3_joint_4: child gen3_forearm_link -> gen3_spherical_wrist_1_link; limit lower=-2.66 upper=2.66 effort=39 velocity=1.3963 -> effort=9 velocity=1.2218; origin xyz=0 0.006375 -0.21038 rpy=1.5708 -6.6954E-17 -1.6653E-16 -> xyz=0 0.20843 -0.006375 rpy=1.5708 0.0 0.0; parent gen3_half_arm_2_link -> gen3_forearm_link; type revolute -> continuous
- joint gen3_joint_5: child gen3_spherical_wrist_1_link -> gen3_spherical_wrist_2_link; limit effort=9 velocity=1.2218 -> lower=-2.09 upper=2.09 effort=9 velocity=1.2218; origin xyz=0 -0.20843 -0.006375 rpy=-1.5708 2.2204E-16 -6.373E-17 -> xyz=0 -0.00017505 -0.10593 rpy=-1.5708 0.0 0.0; parent gen3_forearm_link -> gen3_spherical_wrist_1_link; type continuous -> revolute
- joint gen3_joint_6: child gen3_spherical_wrist_2_link -> gen3_bracelet_link; limit lower=-2.23 upper=2.23 effort=9 velocity=1.2218 -> effort=9 velocity=1.2218; origin xyz=0 0.00017505 -0.10593 rpy=1.5708 9.2076E-28 -8.2157E-15 -> xyz=0 0.10593 -0.00017505 rpy=1.5708 0.0 0.0; parent gen3_spherical_wrist_1_link -> gen3_spherical_wrist_2_link; type revolute -> continuous

Commit message: feat(moveit): MoveIt 2 planifica y burger_kinova_reference valida y ejecuta
move_group se lanza con allow_trajectory_execution: false; la única puerta
hacia el joint_trajectory_controller es el nuevo moveit_safe_executor, que
conserva las salvaguardas validadas en el robot (enable_motion, modo seco,
confirmación, telemetría fresca, límites aprobados, códigos de salida).

burger_kinova_reference:
- trajectory_validation.py: reglas sobre una trayectoria completa
  (arranque en la pose medida, límites, velocidad entre puntos y
  declarada, saltos de 2π en articulaciones continuas, recorrido y
  duración). Lógica pura, 13 pruebas.
- escena_urdf.py + escena_moveit: la mesa de burger_description como
  obstáculo de MoveIt; se niega a cargar si una caja invade la base.
- metas_moveit.py + config/metas_moveit.yaml: metas articulares, poses en
  marcos de burger_description (tag_mesa...), tramos cartesianos y pinza.
- moveit_safe_executor: planifica desde la pose medida (o toma los planes
  del botón Plan de RViz), valida, pide confirmación, ejecuta, cancela si
  la telemetría se pierde y en Ctrl+C, y registra cada plan en JSONL.
- launch/moveit_planificacion.launch.py: move_group sólo planificación,
  RViz y escena; no lanza el driver.

burger_description: table_to_world pasa de z = 0 a z = 0.025 m. Con la
mesa (0.05 m) centrada en table_link, la base del Gen3 quedaba 25 mm
dentro de la mesa y MoveIt declaraba en colisión el estado inicial. Es la
misma altura de tag_mesa.

education: Guía de Laboratorio 04 (Corte 3), Markdown y Word generado con
build_guia_lab_04_moveit2.py.

Co-Authored-By: Claude Opus 5.5 <noreply@anthropic.com>
Claude-Session: https://claude.ai/code/session_01UvpLg8kDntXyQL5Vii4qjP

File: burger_description/urdf/burger_delivery_gen3.urdf (robot description, URDF)
Before this commit: robot burger_delivery_gen3, 45 links, 44 joints
Joints:
- joint table_to_world: origin xyz=0.20 0.30 0.00 rpy=0 0 0 -> xyz=0.20 0.30 0.025 rpy=0 0 0

File: burger_description/urdf/delivery_scene_fixed.urdf (robot description, URDF)
Before this commit: robot burger_delivery_scene, 42 links, 41 joints
Joints:
- joint table_to_world: origin xyz=0.20 0.30 0.00 rpy=0 0 0 -> xyz=0.20 0.30 0.025 rpy=0 0 0

Commit message: fix(burger_description): quitar la cámara de muñeca simulada de Kinova
Los URDF de escena heredaron de ros2_kortex (gen3_2f85.urdf) una cámara
externa tipo RealSense que Kinova usa en Gazebo: la caja
wrist_mounted_camera_link con sus frames de color, profundidad e
infrarrojo, y el soporte wrist_camera_mount_link, una caja de 0,5 kg con
colisión. El Gen3 del laboratorio no tiene esa cámara: su visión está
integrada en el brazalete, ya modelada con bracelet_with_vision_link y
los frames gen3_camera_*.

Se eliminan esos 12 links y sus joints de burger_delivery_gen3.urdf y
delivery_scene_fixed.urdf, y sus entradas de rviz/default.rviz. Ningún
nodo, script ni configuración usaba esos frames.

Verificado: check_urdf en los cuatro URDF; display.launch.py sin
errores; el árbol TF pasa de 56 a 44 frames, sigue conectado con una
sola raíz y conserva gen3_camera_link, gen3_camera_color_frame y
gen3_camera_depth_frame.

Co-Authored-By: Claude Opus 5.5 <noreply@anthropic.com>

File: burger_description/urdf/burger_delivery_gen3.urdf (robot description, URDF)
Before this commit: robot burger_delivery_gen3, 45 links, 44 joints
Links:
- removed link wrist_camera_link
- removed link wrist_camera_mount_link
- removed link wrist_mounted_camera_bottom_screw_frame
- removed link wrist_mounted_camera_color_frame
- removed link wrist_mounted_camera_color_optical_frame
- removed link wrist_mounted_camera_depth_frame
- removed link wrist_mounted_camera_depth_optical_frame
- removed link wrist_mounted_camera_infra1_frame
- removed link wrist_mounted_camera_infra1_optical_frame
- removed link wrist_mounted_camera_infra2_frame
- removed link wrist_mounted_camera_infra2_optical_frame
- removed link wrist_mounted_camera_link
Joints:
- removed joint wrist_camera_joint
- removed joint wrist_camera_mount_joint
- removed joint wrist_mounted_camera_color_joint
- removed joint wrist_mounted_camera_color_optical_joint
- removed joint wrist_mounted_camera_depth_joint
- removed joint wrist_mounted_camera_depth_optical_joint
- removed joint wrist_mounted_camera_infra1_joint
- removed joint wrist_mounted_camera_infra1_optical_joint
- removed joint wrist_mounted_camera_infra2_joint
- removed joint wrist_mounted_camera_infra2_optical_joint
- removed joint wrist_mounted_camera_joint
- removed joint wrist_mounted_camera_link_joint

File: burger_description/urdf/delivery_scene_fixed.urdf (robot description, URDF)
Before this commit: robot burger_delivery_scene, 42 links, 41 joints
Links:
- removed link wrist_camera_link
- removed link wrist_camera_mount_link
- removed link wrist_mounted_camera_bottom_screw_frame
- removed link wrist_mounted_camera_color_frame
- removed link wrist_mounted_camera_color_optical_frame
- removed link wrist_mounted_camera_depth_frame
- removed link wrist_mounted_camera_depth_optical_frame
- removed link wrist_mounted_camera_infra1_frame
- removed link wrist_mounted_camera_infra1_optical_frame
- removed link wrist_mounted_camera_infra2_frame
- removed link wrist_mounted_camera_infra2_optical_frame
- removed link wrist_mounted_camera_link
Joints:
- removed joint wrist_camera_joint
- removed joint wrist_camera_mount_joint
- removed joint wrist_mounted_camera_color_joint
- removed joint wrist_mounted_camera_color_optical_joint
- removed joint wrist_mounted_camera_depth_joint
- removed joint wrist_mounted_camera_depth_optical_joint
- removed joint wrist_mounted_camera_infra1_joint
- removed joint wrist_mounted_camera_infra1_optical_joint
- removed joint wrist_mounted_camera_infra2_joint
- removed joint wrist_mounted_camera_infra2_optical_joint
- removed joint wrist_mounted_camera_joint
- removed joint wrist_mounted_camera_link_joint
